File: doorbellsensor.kicad_pcb (KiCad board)
At the start: 2 copper layers, 49.7 x 49.9 mm, 7 parts, among them J1 Screw_Terminal_01x05, K2 G5V-1-DC5

Commit message: rev 1 - silkscreen improvements
Other:
- board text added: "Rev. 1"
Changed lines of the file:
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@@
 		(tags "THT Terminal Block Phoenix MKDS-1,5-5 pitch 5mm size 25x9.8mm drill 1.3mm pad 2.6mm")
 		(property "Reference" "J1"
-			(at 24 4.5 0)
+			(at -4.075 -0.025 0)
 			(layer "F.SilkS")
 			(effects
@@
 		(tags "Relay Omron G5V-1")
 		(property "Reference" "K2"
-			(at -2.5925 6.4575 180)
+			(at 7.9825 4.9825 180)
 			(layer "F.SilkS")
 			(effects
@@
 		)
 		(property "Value" "G5V-1-DC5"
-			(at 10.9075 4.9575 180)
+			(at -2.5175 4.9825 180)
 			(layer "F.SilkS")
 			(effects
@@
 		(tags "CP Radial series Radial pin pitch 2.50mm diameter 5mm height 7mm Electrolytic Capacitor")
 		(property "Reference" "C1"
-			(at 3 -3.5 180)
+			(at 1.975 4.075 180)
 			(layer "F.SilkS")
 			(effects
@@
 		)
 		(property "Value" "22 uF"
-			(at 6.5 -2 0)
+			(at 0.475 -3.925 0)
 			(layer "F.SilkS")
 			(effects
@@
 		(tags "Diode DO-41_SOD81 series Axial Horizontal pin pitch 10.16mm  length 5.2mm diameter 2.7mm")
 		(property "Reference" "D1"
-			(at 5.08 2.5 0)
+			(at 5.08 -2.575 0)
 			(layer "F.SilkS")
 			(effects
@@
 		)
 		(property "Value" "1N4003"
-			(at 5.08 -2.5 0)
+			(at 5.105 2.925 0)
 			(layer "F.SilkS")
 			(effects
@@
 	)
 	(gr_text "1"
-		(at 100.5 130 0)
+		(at 99.525 131.925 0)
 		(layer "F.SilkS")
 		(effects
 			(font
-				(size 1 1)
-				(thickness 0.1)
+				(size 2.032 2.032)
+				(thickness 0.254)
 			)
 			(justify left bottom)
@@
 	)
 	(gr_text "NC"
-		(at 100 115 0)
+		(at 98.025 116.425 0)
+		(layer "F.SilkS")
+		(effects
+			(font
+				(size 2.032 2.032)
+				(thickness 0.254)
+			)
+			(justify left bottom)
+		)
+	)
+	(gr_text "NO"
+		(at 98.025 121.425 0)
+		(layer "F.SilkS")
+		(effects
+			(font
+				(size 2.032 2.032)
+				(thickness 0.254)
+			)
+			(justify left bottom)
+		)
+	)
+	(gr_text "Rev. 1"
+		(at 101.525 146.425 0)
 		(layer "F.SilkS")
 		(effects
@@
 		)
 	)
-	(gr_text "NO"
-		(at 100 120 0)
+	(gr_text "C"
+		(at 99.025 126.925 0)
 		(layer "F.SilkS")
 		(effects
 			(font
-				(size 1 1)
-				(thickness 0.1)
+				(size 2.032 2.032)
+				(thickness 0.254)
 			)
 			(justify left bottom)
 		)
 	)
-	(gr_text "C"
-		(at 100.5 125 0)
+	(gr_text "X"
+		(at 99.525 136.925 0)
 		(layer "F.SilkS")
 		(effects
 			(font
-				(size 1 1)
-				(thickness 0.1)
+				(size 2.032 2.032)
+				(thickness 0.254)
 			)
 			(justify left bottom)
-		)
-	)
-	(gr_text "X"
-		(at 100.5 135 0)
-		(layer "F.SilkS")
-		(effects
-			(font
-				(size 1 1)
-				(thickness 0.1)
-			)
-			(justify left bottom)
